File: Hardware/Radio.kicad_sch (KiCad schematic)
At the start: 17 parts, among them J1 3.5 mm Mono Audio Jack, SW1 Switch, U1 LM386

Commit message: Add files via upload
Parts:
- R1: value 10k -> 10
Changed lines of the file:
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@@
 			)
 		)
-		(property "Value" "10k"
+		(property "Value" "10"
 			(at 179.07 107.9499 0)
 			(show_name no)
